File: hardware/pcb/esp32_athan.kicad_sch (KiCad schematic)
At the start: 39 parts, among them J1 USB_C_Receptacle_PowerOnly_6P, J2 Barrel_Jack, J3 Speaker, J5 Relay, J6 PROG, U1 ESP32-S3-WROOM-1-N16R8, U2 SKQUAAA010, U3 AMS1117-3.3, U4 MAX98357A

Commit message: USB-C on either side, switch named by its real part, STEP out of the repo
Board
- J1 has a new footprint, USB_C_Receptacle_GCT_USB4125_6P_BothSides
  (project library): KiCad's GCT USB4125 with its six pads also on the
  back, the four shell legs in shared holes. The receptacle can be
  soldered on the front by hand or placed on the back by JLCPCB. Flipped
  onto the back, its A and B pins land on each other's pads: CC1 and CC2
  swap (each has its own 4.7 kΩ), VBUS and GND stay on their nets.
- Copper at J1 rearranged for the back pads: the two +5V vias moved
  1.1 mm right, VBUS pads on both sides tracked to them, and two vias take
  the back CC pads to the front lines to R1 and R2.
- A +3V3 track on the back near U4 is now two 0.6 mm segments.
- U2 is named for the switch it is: "5-way switch (SKQUCAA010 type)",
  a 10 x 10 mm through-hole 5-way switch with a centre push (Alps
  SKQUCAA010 or a copy). Its description warns that Alps' SKQUAAA010,
  which fits the same holes, has no centre push. SnapEDA's shop links
  for SKQUAAA010 are removed; the pins and footprint are unchanged.
- Checks: DRC 0 errors, 0 unconnected, schematic and board match, ERC 0
  errors.

JLCPCB files
- jlcpcb_assembly.py places a part whose footprint has pads on both
  sides on the side the selection file names ("sides", the back by
  default), as the same part flipped over. --verify checks it against
  JLCPCB's footprint like every other part: J1 on the back fits within
  0.075 mm.
- jlcpcb_select.py draws J1 on both sides (dotted blue where it is not
  fitted); a click on the other side moves it there. The choice is saved
  in jlcpcb_selection.json, now J1 on the back.
- generate_fab_files.sh notes J1's side in fab_files/README.md.
- J1 joins the back-only order: three extended parts there (U1, U4, J1).
Parts:
- J1: footprint Connector_USB:USB_C_Receptacle_GCT_USB4125-xx-x_6P_TopMnt_Horizontal -> Library:USB_C_Receptacle_GCT_USB4125_6P_BothSides
- U2: value SKQUAAA010 -> 5-way switch (SKQUCAA010 type); Availability In Stock -> (none); Check_prices https://www.snapeda.com/parts/SKQUAAA010/ALPS/view-part/?re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 -> (none); MP SKQUAAA010 -> SKQUCAA010; Package None -> (none); Price None -> (none); Purchase-URL https://www.snapeda.com/api/url_track_click_mouser/?unipart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 -> (none); SnapEDA_Link https://www.snapeda.com/parts/SKQUAAA010/ALPS/view-part/?re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 -> (none)
Changed lines of the file:
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@@
 			)
 		)
-		(property "Footprint" "Connector_USB:USB_C_Receptacle_GCT_USB4125-xx-x_6P_TopMnt_Horizontal"
+		(property "Footprint" "Library:USB_C_Receptacle_GCT_USB4125_6P_BothSides"
 			(at 50.8 53.34 0)
 			(hide yes)
@@
 			)
 		)
-		(property "Description" "USB-C power input, 5 V (power only, no data)"
+		(property "Description" "USB-C power input, 5 V (power only, no data); fits on the front or the back"
 			(at 46.99 55.88 0)
 			(hide yes)
@@
 			)
 		)
-		(property "Value" "SKQUAAA010"
+		(property "Value" "5-way switch (SKQUCAA010 type)"
 			(at 144.78 167.6399 0)
 			(show_name no)
@@
 			)
 		)
-		(property "Description" "5-way switch (4 directions and a centre push), Alps SKQUAAA010, through-hole"
+		(property "Description" "5-way switch, 10 x 10 mm through-hole, 4 directions and a centre push: Alps SKQUCAA010 or a copy (sold as 5-way switch 10*10*10 mm). Not SKQUAAA010, which has no centre push"
 			(at 146.05 158.75 0)
 			(hide yes)
@@
 			)
 		)
-		(property "Package" "None"
-			(at 146.05 158.75 0)
-			(hide yes)
-			(show_name no)
-			(do_not_autoplace no)
-			(effects
-				(font
-					(size 1.27 1.27)
-				)
-				(justify bottom)
-			)
-		)
-		(property "Price" "None"
-			(at 146.05 158.75 0)
-			(hide yes)
-			(show_name no)
-			(do_not_autoplace no)
-			(effects
-				(font
-					(size 1.27 1.27)
-				)
-				(justify bottom)
-			)
-		)
-		(property "SnapEDA_Link" "https://www.snapeda.com/parts/SKQUAAA010/ALPS/view-part/?ref=snap"
-			(at 146.05 158.75 0)
-			(hide yes)
-			(show_name no)
-			(do_not_autoplace no)
-			(effects
-				(font
-					(size 1.27 1.27)
-				)
-				(justify bottom)
-			)
-		)
-		(property "MP" "SKQUAAA010"
-			(at 146.05 158.75 0)
-			(hide yes)
-			(show_name no)
-			(do_not_autoplace no)
-			(effects
-				(font
-					(size 1.27 1.27)
-				)
-				(justify bottom)
-			)
-		)
-		(property "Purchase-URL" "https://www.snapeda.com/api/url_track_click_mouser/?unipart_id=104101&manufacturer=ALPS&part_name=SKQUAAA010&search_term=skquaaa010"
-			(at 146.05 158.75 0)
-			(hide yes)
-			(show_name no)
-			(do_not_autoplace no)
-			(effects
-				(font
-					(size 1.27 1.27)
-				)
-				(justify bottom)
-			)
-		)
-		(property "Availability" "In Stock"
-			(at 146.05 158.75 0)
-			(hide yes)
-			(show_name no)
-			(do_not_autoplace no)
-			(effects
-				(font
-					(size 1.27 1.27)
-				)
-				(justify bottom)
-			)
-		)
-		(property "Check_prices" "https://www.snapeda.com/parts/SKQUAAA010/ALPS/view-part/?ref=eda"
+		(property "MP" "SKQUCAA010"
 			(at 146.05 158.75 0)
 			(hide yes)
